File: MPPT_PCB rev8/MPPT/MPPT.kicad_sch (KiCad schematic)
At the start: 6 parts

Commit message: PCB (#98)
Parts:
- gave numbers to parts that had none: 6
Connections:
- net at Q2.1 (G), Q3.1 (G): now also Q4.1 (G), U1.2
Changed lines of the file:
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@@
   (junction (at 88.9 81.28) (diameter 0) (color 0 0 0 0)
+  )
+  (junction (at 53.34 40.64) (diameter 0) (color 0 0 0 0)
+  )
+  (junction (at 81.28 76.2) (diameter 0) (color 0 0 0 0)
   )
   (junction (at 88.9 71.12) (diameter 0) (color 0 0 0 0)
@@
     (stroke (width 0) (type default) (color 0 0 0 0))
   )
+  (wire (pts (xy 124.46 27.94) (xy 53.34 27.94))
+    (stroke (width 0) (type default) (color 0 0 0 0))
+  )
   (wire (pts (xy 132.08 33.02) (xy 132.08 38.1))
+    (stroke (width 0) (type default) (color 0 0 0 0))
+  )
+  (wire (pts (xy 53.34 27.94) (xy 53.34 40.64))
     (stroke (width 0) (type default) (color 0 0 0 0))
   )
@@
     (stroke (width 0) (type default) (color 0 0 0 0))
   )
+  (wire (pts (xy 53.34 76.2) (xy 53.34 40.64))
+    (stroke (width 0) (type default) (color 0 0 0 0))
+  )
   (wire (pts (xy 88.9 48.26) (xy 88.9 71.12))
+    (stroke (width 0) (type default) (color 0 0 0 0))
+  )
+  (wire (pts (xy 81.28 76.2) (xy 53.34 76.2))
     (stroke (width 0) (type default) (color 0 0 0 0))
   )
@@
     (stroke (width 0) (type default) (color 0 0 0 0))
   )
+  (wire (pts (xy 124.46 43.18) (xy 124.46 27.94))
+    (stroke (width 0) (type default) (color 0 0 0 0))
+  )
   (symbol (lib_id "Transistor_FET:IRLZ44N") (at 86.36 76.2 0) (unit 1)
     (in_bom yes) (on_board yes) (fields_autoplaced)
-    (property "Reference" "Q?" (id 0) (at 92.71 74.9299 0)
+    (property "Reference" "Q2" (id 0) (at 92.71 74.9299 0)
       (effects (font (size 1.27 1.27)) (justify left))
     )
@@
   (symbol (lib_id "Transistor_FET:IRLZ44N") (at 86.36 43.18 0) (unit 1)
     (in_bom yes) (on_board yes) (fields_autoplaced)
-    (property "Reference" "Q?" (id 0) (at 92.71 41.9099 0)
+    (property "Reference" "Q1" (id 0) (at 92.71 41.9099 0)
       (effects (font (size 1.27 1.27)) (justify left))
     )
@@
   (symbol (lib_id "74xx:74AHC04") (at 45.72 40.64 0) (unit 1)
     (in_bom yes) (on_board yes) (fields_autoplaced)
-    (property "Reference" "U?" (id 0) (at 45.72 31.75 0))
+    (property "Reference" "U1" (id 0) (at 45.72 31.75 0))
     (property "Value" "74AHC04" (id 1) (at 45.72 34.29 0))
     (property "Footprint" "" (id 2) (at 45.72 40.64 0)
@@
   (symbol (lib_id "Transistor_FET:IRLZ44N") (at 129.54 76.2 0) (unit 1)
     (in_bom yes) (on_board yes) (fields_autoplaced)
-    (property "Reference" "Q?" (id 0) (at 135.89 74.9299 0)
+    (property "Reference" "Q5" (id 0) (at 135.89 74.9299 0)
       (effects (font (size 1.27 1.27)) (justify left))
     )
@@
   (symbol (lib_id "Transistor_FET:IRLZ44N") (at 129.54 43.18 0) (unit 1)
     (in_bom yes) (on_board yes) (fields_autoplaced)
-    (property "Reference" "Q?" (id 0) (at 135.89 41.9099 0)
+    (property "Reference" "Q4" (id 0) (at 135.89 41.9099 0)
       (effects (font (size 1.27 1.27)) (justify left))
     )
@@
   (symbol (lib_id "Transistor_FET:IRLZ44N") (at 86.36 76.2 0) (unit 1)
     (in_bom yes) (on_board yes) (fields_autoplaced)
-    (property "Reference" "Q?" (id 0) (at 92.71 74.9299 0)
+    (property "Reference" "Q3" (id 0) (at 92.71 74.9299 0)
       (effects (font (size 1.27 1.27)) (justify left))
     )
@@
   )
   (symbol_instances
+    (path "/21b332fe-4f14-42c5-abdd-64b17be8e6c4"
+      (reference "Q1") (unit 1) (value "IRLZ44N") (footprint "Package_TO_SOT_THT:TO-220-3_Vertical")
+    )
     (path "/17ae4327-88f5-4ed5-ba12-7ad5a46f57b2"
-      (reference "Q?") (unit 1) (value "IRLZ44N") (footprint "Package_TO_SOT_THT:TO-220-3_Vertical")
+      (reference "Q2") (unit 1) (value "IRLZ44N") (footprint "Package_TO_SOT_THT:TO-220-3_Vertical")
     )
-    (path "/21b332fe-4f14-42c5-abdd-64b17be8e6c4"
-      (reference "Q?") (unit 1) (value "IRLZ44N") (footprint "Package_TO_SOT_THT:TO-220-3_Vertical")
+    (path "/c993d47e-0704-45fd-8f9f-89195a95f9f4"
+      (reference "Q3") (unit 1) (value "IRLZ44N") (footprint "Package_TO_SOT_THT:TO-220-3_Vertical")
+    )
+    (path "/a72eb2dc-204b-45da-8fb7-9ab252d6ddda"
+      (reference "Q4") (unit 1) (value "IRLZ44N") (footprint "Package_TO_SOT_THT:TO-220-3_Vertical")
     )
     (path "/a21d5cc9-8637-46c9-9b58-7bc2b70bcb0a"
-      (reference "Q?") (unit 1) (value "IRLZ44N") (footprint "Package_TO_SOT_THT:TO-220-3_Vertical")
-    )
-    (path "/a72eb2dc-204b-45da-8fb7-9ab252d6ddda"
-      (reference "Q?") (unit 1) (value "IRLZ44N") (footprint "Package_TO_SOT_THT:TO-220-3_Vertical")
-    )
-    (path "/c993d47e-0704-45fd-8f9f-89195a95f9f4"
-      (reference "Q?") (unit 1) (value "IRLZ44N") (footprint "Package_TO_SOT_THT:TO-220-3_Vertical")
+      (reference "Q5") (unit 1) (value "IRLZ44N") (footprint "Package_TO_SOT_THT:TO-220-3_Vertical")
     )
     (path "/4a992c7a-278b-4097-b1fa-0edf145bf298"
-      (reference "U?") (unit 1) (value "74AHC04") (footprint "")
+      (reference "U1") (unit 1) (value "74AHC04") (footprint "")
     )
   )
